Commit message: - Added cylinder inertia for wheels, box for body

File: pinpointbot_description/urdf/pinpoint_include.xacro (robot description, xacro)
@@ -1,3 +1,36 @@
 <?xml version="1.0"?>
 <robot xmlns:xacro="http://www.ros.org/wiki/xacro">
+<!-- =============== Inertia macros ==============-->
+<!-- Based on https://en.wikipedia.org/wiki/List_of_moments_of_inertia -->
+<!-- https://github.com/ros-mobile-robots/mobile_robot_description/blob/48819dcec6f897b7d02e8d4aa6c66d803ddf6239/urdf/include/common_macros.urdf.xacro -->
+<!--
+  params:
+  - m [float]: link mass;
+  - r [float]: cylinder radius;
+  - l [float]: cylinder lenght (height);
+-->
+  <xacro:macro name="cylinder_inertia" params="m r l o_xyz:='0.0 0.0 0.0' o_rpy:='0.0 0.0 0.0'">
+    <inertial>
+      <mass value="${m}"/>
+      <inertia ixx="${m*(3*r*r+l*l)/12}" ixy = "0" ixz = "0"
+               iyy="${m*(3*r*r+l*l)/12}" iyz = "0" izz="${m*r*r/2}"/>
+      <origin xyz="${o_xyz}" rpy="${o_rpy}" />
+    </inertial>
+  </xacro:macro>
+<!--
+  params:
+  - m [float]: link mass;
+  - x [float]: link dimension on the X-axis;
+  - y [float]: link dimension on the Y-axis;
+  - z [float]: link dimension on the Z-axis;
+-->
+ <xacro:macro name="box_inertia" params="m x y z o_xyz:='0.0 0.0 0.0' o_rpy:='0.0 0.0 0.0'">
+    <inertial>
+      <mass value="${m}"/>
+      <inertia ixx="${m / 12.0 * (y*y + z*z)}" ixy="0.0" ixz="0.0"
+               iyy="${m / 12.0 * (x*x + z*z)}" iyz="0.0"
+               izz="${m / 12.0 * (x*x + y*y)}"/>
+      <origin xyz="${o_xyz}" rpy="${o_rpy}" />
+    </inertial>
+  </xacro:macro>
 </robot>

Commit message: - Added sphere inertia

File: pinpointbot_description/urdf/pinpoint_include.xacro (robot description, xacro)
@@ -34,3 +34,14 @@
     </inertial>
   </xacro:macro>
+<!--
+  params:
+  - m [float]: link mass;
+  - r [float]: sphere radius;
+-->
+  <xacro:macro name="sphere_inertia" params="m r">
+    <inertial>
+      <mass value="${m}"/>
+      <inertia ixx="${2.0*m*(r*r)/5.0}" ixy="0.0" ixz="0.0" iyy="${2.0*m*(r*r)/5.0}" iyz="0.0" izz="${2.0*m*(r*r)/5.0}"/>
+    </inertial>
+  </xacro:macro>
 </robot>
